File: hardware/rev1.3/connectors.sch (KiCad schematic (older format))
At the start: 4 parts, among them J1 Conn_02x05_Odd_Even, J2 Arduino_UNO_R3, J3 Conn_02x14_Top_Bottom, J4 Conn_02x14_Top_Bottom

Commit message: Upgrade to KiCad 5.1.x
Parts:
- J1: symbol Connector:Conn_02x05_Odd_Even -> main-rescue:Conn_02x05_Odd_Even-Connector
- J2: symbol modules:Arduino_UNO_R3 -> main-rescue:Arduino_UNO_R3-modules
- J3, J4: symbol Connector:Conn_02x14_Odd_Even -> main-rescue:Conn_02x14_Odd_Even-Connector
Changed lines of the file:
@@
 EESchema Schematic File Version 4
 LIBS:main-cache
-EELAYER 26 0
+EELAYER 29 0
 EELAYER END
 $Descr A4 11693 8268
@@
 $EndDescr
 $Comp
-L Connector:Conn_02x05_Odd_Even J1
+L main-rescue:Conn_02x05_Odd_Even-Connector J1
 U 1 1 5B75812E
 P 1750 1300
+AR Path="/5B75812E" Ref="J1"  Part="1"
+AR Path="/5B74872F/5B75812E" Ref="J1"  Part="1"
 F 0 "J1" H 1800 1300 50  0000 C CNN
 F 1 "Conn_02x05_Odd_Even" H 1800 1626 50  0001 C CNN
@@
 	1850 850  1800 850
 $Comp
-L Connector:Conn_02x14_Odd_Even J3
+L main-rescue:Conn_02x14_Odd_Even-Connector J3
 U 1 1 5B760B19
 P 4200 2750
@@
 $EndComp
 $Comp
-L Connector:Conn_02x14_Odd_Even J4
+L main-rescue:Conn_02x14_Odd_Even-Connector J4
 U 1 1 5B760B20
 P 6000 2750
@@
 $EndComp
 $Comp
-L modules:Arduino_UNO_R3 J2
+L main-rescue:Arduino_UNO_R3-modules J2
 U 1 1 5B760B27
 P 2100 2750
