File: hardware/rev1.3/crystals.sch (KiCad schematic (older format))
At the start: 6 parts, among them Y1 16 MHz, Y2 32768

Commit message: Upgrade to KiCad 5.1.x
Parts:
- C1, C2, C3, C4: symbol device:C -> main-rescue:C-device
- Y1, Y2: symbol device:Crystal -> main-rescue:Crystal-device
Changed lines of the file:
@@
 EESchema Schematic File Version 4
 LIBS:main-cache
-EELAYER 26 0
+EELAYER 29 0
 EELAYER END
 $Descr A4 11693 8268
@@
 $EndComp
 $Comp
-L device:C C2
+L main-rescue:C-device C2
 U 1 1 5B7344A6
 P 1250 1450
@@
 $EndComp
 $Comp
-L device:C C1
+L main-rescue:C-device C1
 U 1 1 5B7344AD
 P 800 1450
@@
 $EndComp
 $Comp
-L device:Crystal Y1
+L main-rescue:Crystal-device Y1
 U 1 1 5B7344B4
 P 1050 1100
@@
 $EndComp
 $Comp
-L device:C C4
+L main-rescue:C-device C4
 U 1 1 5B745910
 P 2200 1450
@@
 $EndComp
 $Comp
-L device:C C3
+L main-rescue:C-device C3
 U 1 1 5B745917
 P 1750 1450
@@
 $EndComp
 $Comp
-L device:Crystal Y2
+L main-rescue:Crystal-device Y2
 U 1 1 5B74591E
 P 2000 1100
