File: hardware/rev1.3/main.sch (KiCad schematic (older format))
At the start: 6 parts

Commit message: Upgrade to KiCad 5.1.x
Parts:
- MK1, MK2, MK3, MK4: symbol Mechanical:Mounting_Hole -> main-rescue:Mounting_Hole-Mechanical
Changed lines of the file:
@@
 EESchema Schematic File Version 4
 LIBS:main-cache
-EELAYER 26 0
+EELAYER 29 0
 EELAYER END
 $Descr A4 11693 8268
@@
 $EndSheet
 $Comp
-L Mechanical:Mounting_Hole MK1
+L main-rescue:Mounting_Hole-Mechanical MK1
 U 1 1 5B07E576
 P 3150 950
@@
 $EndComp
 $Comp
-L Mechanical:Mounting_Hole MK2
+L main-rescue:Mounting_Hole-Mechanical MK2
 U 1 1 5B07E86F
 P 3150 1100
@@
 $EndComp
 $Comp
-L Mechanical:Mounting_Hole MK3
+L main-rescue:Mounting_Hole-Mechanical MK3
 U 1 1 5B07E889
 P 3150 1250
@@
 $EndComp
 $Comp
-L Mechanical:Mounting_Hole MK4
+L main-rescue:Mounting_Hole-Mechanical MK4
 U 1 1 5B07E8A5
 P 3150 1400
