File: hardware/rev1.3/mcu.sch (KiCad schematic (older format))
At the start: 12 parts, among them SW1 FSM1LP, SW2 FSM1LP, U1 STM32F405RGTx

Commit message: Upgrade to KiCad 5.1.x
Parts:
- C10, C11, C12, C13: symbol device:C -> main-rescue:C-device
- D2: symbol device:LED -> main-rescue:LED-device
- JP1, JP2: symbol device:Jumper -> main-rescue:Jumper-device
- R2, R3: symbol device:R -> main-rescue:R-device
- U1: symbol MCU_ST_STM32:STM32F405RGTx -> main-rescue:STM32F405RGTx-MCU_ST_STM32
Changed lines of the file:
@@
 EESchema Schematic File Version 4
 LIBS:main-cache
-EELAYER 26 0
+EELAYER 29 0
 EELAYER END
 $Descr A4 11693 8268
@@
 $EndDescr
 $Comp
-L MCU_ST_STM32:STM32F405RGTx U?
+L main-rescue:STM32F405RGTx-MCU_ST_STM32 U?
 U 1 1 5B07CDF0
 P 6100 4050
@@
 Connection ~ 6000 1950
 $Comp
-L device:C C10
+L main-rescue:C-device C10
 U 1 1 5B07CE17
 P 1150 3200
@@
 $EndComp
 $Comp
-L device:Jumper JP1
+L main-rescue:Jumper-device JP1
 U 1 1 5B07CE24
 P 1400 2650
@@
 	1700 2450 1800 2450
 $Comp
-L device:C C11
+L main-rescue:C-device C11
 U 1 1 5B07CE46
 P 1400 1850
@@
 PD2
 $Comp
-L device:LED D2
+L main-rescue:LED-device D2
 U 1 1 5B07CE5B
 P 2500 1550
@@
 $EndComp
 $Comp
-L device:R R2
+L main-rescue:R-device R2
 U 1 1 5B07CE62
 P 2950 1550
@@
 	1800 5650 1550 5650
 $Comp
-L device:C C12
+L main-rescue:C-device C12
 U 1 1 5B0728D5
 P 1600 3200
@@
 	1150 3400 1150 3350
 $Comp
-L device:Jumper JP2
+L main-rescue:Jumper-device JP2
 U 1 1 5B307112
 P 4700 1650
@@
 	4300 1650 4400 1650
 $Comp
-L device:C C13
+L main-rescue:C-device C13
 U 1 1 5B30712E
 P 4000 1050
@@
 Connection ~ 4300 1500
 $Comp
-L device:R R3
+L main-rescue:R-device R3
 U 1 1 5B30A9BB
 P 4300 900
