File: hardware/rev1.3/power.sch (KiCad schematic (older format))
At the start: 8 parts

Commit message: Upgrade to KiCad 5.1.x
Parts:
- BT1: symbol device:Battery_Cell -> main-rescue:Battery_Cell-device
- C5, C6, C7, C8, C9: symbol device:C -> main-rescue:C-device
- D1: symbol device:LED -> main-rescue:LED-device
- R1: symbol device:R -> main-rescue:R-device
Changed lines of the file:
@@
 EESchema Schematic File Version 4
 LIBS:main-cache
-EELAYER 26 0
+EELAYER 29 0
 EELAYER END
 $Descr A4 11693 8268
@@
 $EndComp
 $Comp
-L device:C C5
+L main-rescue:C-device C5
 U 1 1 5B06DF0F
 P 800 1050
@@
 Connection ~ 1800 850
 $Comp
-L device:C C6
+L main-rescue:C-device C6
 U 1 1 5B06DF30
 P 1150 1050
@@
 $EndComp
 $Comp
-L device:C C7
+L main-rescue:C-device C7
 U 1 1 5B06DF37
 P 1500 1050
@@
 $EndComp
 $Comp
-L device:C C8
+L main-rescue:C-device C8
 U 1 1 5B06DF3E
 P 1800 1050
@@
 $EndComp
 $Comp
-L device:C C9
+L main-rescue:C-device C9
 U 1 1 5B06DF45
 P 2150 1050
@@
 $EndComp
 $Comp
-L device:Battery_Cell BT1
+L main-rescue:Battery_Cell-device BT1
 U 1 1 5B06DF4C
 P 2850 1150
@@
 $EndComp
 $Comp
-L device:LED D1
+L main-rescue:LED-device D1
 U 1 1 5B0710EF
 P 1150 2000
@@
 $EndComp
 $Comp
-L device:R R1
+L main-rescue:R-device R1
 U 1 1 5B0710F6
 P 1600 2000
